File: pcb/keystation/key.kicad_sch (KiCad schematic)
At the start: 15 parts, among them J1 Button, Q1 IRF540N, U1 ATtiny84A-CC, U2 LM741, U3 LM1117MP-3.3

Commit message: keystation pcb
Parts:
- removed U1: ATtiny84A-CC, Package_BGA:UFBGA-15_3.0x3.0mm_Layout4x4_P0.65mm, symbol MCU_Microchip_ATtiny:ATtiny84A-CC
- added D1: MBR0520, Diode_SMD:D_SOD-123, symbol Diode:MBR0520
- added J2: speaker, Connector_Molex:Molex_KK-254_AE-6410-02A_1x02_P2.54mm_Vertical, symbol Connector_Generic:Conn_01x02
- added J3: Vin, Connector_Molex:Molex_KK-254_AE-6410-02A_1x02_P2.54mm_Vertical, symbol Connector_Generic:Conn_01x02
- added J4: AVR-ISP-6, Connector_IDC:IDC-Header_2x03_P2.54mm_Vertical, symbol Connector:AVR-ISP-6
- added R3: 1k, Resistor_SMD:R_0805_2012Metric_Pad1.20x1.40mm_HandSolder, symbol Device:R
- added R4: 10k, Resistor_SMD:R_0805_2012Metric_Pad1.20x1.40mm_HandSolder, symbol Device:R
- added U4: ATtiny84A-SS, Package_SO:SOIC-14_3.9x8.7mm_P1.27mm, symbol MCU_Microchip_ATtiny:ATtiny84A-SS
- C1, C2, C3: footprint (none) -> Capacitor_SMD:C_0805_2012Metric_Pad1.18x1.45mm_HandSolder
- Gate-bias1: renamed from Gate-bias; footprint (none) -> Resistor_SMD:R_0805_2012Metric_Pad1.20x1.40mm_HandSolder
- J1: footprint (none) -> Connector_Molex:Molex_KK-254_AE-6410-02A_1x02_P2.54mm_Vertical
- PressureSensor1: renamed from PressureSensor; footprint (none) -> Resistor_SMD:R_0805_2012Metric_Pad1.20x1.40mm_HandSolder
- Pulldown1: renamed from Pulldown; footprint (none) -> Resistor_SMD:R_0805_2012Metric_Pad1.20x1.40mm_HandSolder
- R1, R2: footprint (none) -> Resistor_SMD:R_0805_2012Metric_Pad1.20x1.40mm_HandSolder
- RM1: renamed from RM; footprint (none) -> Resistor_SMD:R_0805_2012Metric_Pad1.20x1.40mm_HandSolder
- U2: footprint (none) -> Package_DIP:DIP-8_W7.62mm_Socket_LongPads
Connections:
- net SPIMISO to controller is gone; now on net MISO: DWM1.19 (SPIMISO)
- net SPIMOSI from controller is gone; now on net MOSI: DWM1.18 (SPIMOSI)
- net +3.3V: now also C2.1, D1.1 (K), R4.1, U4.1 (VCC); no longer C2.2
- net GND: now also C2.2, DWM1.2 (WAKEUP), J2.2 (Pin_2), J3.1 (Pin_1), J4.6 (GND), U4.14 (GND); no longer C2.1
- net MISO: now also J4.1 (MISO), U4.8 (PA5)
- net MOSI: now also J4.4 (MOSI), U4.7 (PA6)
- net alarm: now also R3.1, U4.11 (PA2)
- net button: now also U4.10 (PA3)
- net confirmation: now also U4.12 (PA1)
- net +12V: no longer names the net of C1.1, U3.3 (VI)
- net +12V: now also J3.2 (Pin_2)
- net DWM_RSTn renamed RST
- net RST: now also J4.5 (~{RST}), R4.2, U4.4 (~{RESET}/PB3)
- net SPI mode selector: no longer names the net of DWM1.10 (GPIO5/EXTTXE/SPIPOL)
- net SPI mode selector: no longer DWM1.9 (GPIO6/EXTRXE/SPIHA)
- net SPICLK from controller renamed SCK
- net SCK: now also J4.3 (SCK), U4.9 (PA4)
- net SPICSn from controller renamed Csn
- net Csn: now also U4.6 (PA7)
- new net: D1.2 (A), J4.2 (VCC)
- new net: J2.1 (Pin_1), R3.2
- no-connect marks 0 -> 13
Other:
- note added: "ISP"
- moved on the sheet: DWM1, R1

Commit message: update pcb
Parts:
- added D2, D3, D4, D5: LED, LED_SMD:LED_0805_2012Metric_Pad1.15x1.40mm_HandSolder, symbol Device:LED
Connections:
- net GND: now also D2.1 (K), D3.1 (K), D4.1 (K), D5.1 (K)
- net alarm: now also D3.2 (A)
- net button: now also D4.2 (A)
- net confirmation: now also D2.2 (A)
- net at DWM1.11 (GPIO4/EXTPA): now also D5.2 (A)
- no-connect marks 13 -> 12

Commit message: dish pcb updated
Parts:
- removed D2, D3, D4, D5: LED, LED_SMD:LED_0805_2012Metric_Pad1.15x1.40mm_HandSolder, symbol Device:LED
- removed J3: Vin, Connector_Molex:Molex_KK-254_AE-6410-02A_1x02_P2.54mm_Vertical, symbol Connector_Generic:Conn_01x02
- removed R3: 1k, Resistor_SMD:R_0805_2012Metric_Pad1.20x1.40mm_HandSolder, symbol Device:R
- removed U4: ATtiny84A-SS, Package_SO:SOIC-14_3.9x8.7mm_P1.27mm, symbol MCU_Microchip_ATtiny:ATtiny84A-SS
- added C4: 1uF, Capacitor_SMD:C_0805_2012Metric_Pad1.18x1.45mm_HandSolder, symbol Device:C
- added C5, C6: 22p, Capacitor_SMD:C_0805_2012Metric_Pad1.18x1.45mm_HandSolder, symbol Device:C
- added J5: Conn_01x08, Connector_Molex:Molex_KK-254_AE-6410-08A_1x08_P2.54mm_Vertical, symbol Connector_Generic:Conn_01x08
- added J6: Barrel_Jack_Switch, Connector_BarrelJack:BarrelJack_CUI_PJ-102AH_Horizontal, symbol Connector:Barrel_Jack_Switch
- added U1: ATmega328-A, Package_QFP:TQFP-32_7x7mm_P0.8mm, symbol MCU_Microchip_ATmega:ATmega328-A
- added Y1: 16MHz, Crystal:Crystal_HC49-U_Vertical, symbol Device:Crystal
Connections:
- net +3.3V: now also C4.2, U1.18 (AVCC), U1.4 (VCC), U1.6 (VCC)
- net Csn: now also J5.8 (Pin_8)
- net GND: now also C4.1, C5.2, C6.2, J6.1, J6.2, U1.21 (GND), U1.3 (GND), U1.5 (GND)
- net MISO: now also J5.5 (Pin_5), U1.16 (PB4)
- net MOSI: now also J5.4 (Pin_4), U1.15 (PB3)
- net SCK: now also J5.6 (Pin_6), U1.17 (PB5)
- net alarm: now also J2.1 (Pin_1), J5.3 (Pin_3), U1.14 (PB2)
- net button: now also J5.2 (Pin_2), U1.13 (PB1)
- net confirmation: now also J5.1 (Pin_1), U1.12 (PB0)
- net at C1.1, U3.3 (VI): now also J6.3
- net RST renamed RESET
- net RESET: now also J5.7 (Pin_7), U1.29 (~{RESET}/PC6)
- net interrupt: no longer names the net of DWM1.22 (IRQ/GPIO8), R1.2
- new net: C6.1, U1.7 (XTAL1/PB6), Y1.2
- new net: C5.1, U1.8 (XTAL2/PB7), Y1.1
- no-connect marks 12 -> 27
