File: pcb/keychain/keychain.kicad_pcb (KiCad board)
At the start: 2 copper layers, 43.2 x 30.5 mm, 10 parts, among them J2 AVR-ISP-6, J3 Vin, U1 ATtiny84A-SS, U3 LM1117MP-3.3

Commit message: update pcb
Parts:
- added D2: LED, LED_SMD:LED_0805_2012Metric_Pad1.15x1.40mm_HandSolder, F.Cu at (149.9, 81.3)
Connections:
- DWM1 pad 11: unconnected-(DWM1-GPIO4/EXTPA-Pad11) -> Net-(D2-A)
Routing:
- net Net-(D2-A): track 0.00 -> 26.8 mm
Changed lines of the file:
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@@
   (net 8 "unconnected-(DWM1-GPIO6{slash}EXTRXE{slash}SPIHA-Pad9)")
   (net 9 "unconnected-(DWM1-GPIO5{slash}EXTTXE{slash}SPIPOL-Pad10)")
-  (net 10 "unconnected-(DWM1-GPIO4{slash}EXTPA-Pad11)")
+  (net 10 "Net-(D2-A)")
   (net 11 "unconnected-(DWM1-GPIO3{slash}TXLED-Pad12)")
   (net 12 "unconnected-(DWM1-GPIO2{slash}RXLED-Pad13)")
@@
       (net 9 "unconnected-(DWM1-GPIO5{slash}EXTTXE{slash}SPIPOL-Pad10)") (pinfunction "GPIO5/EXTTXE/SPIPOL") (pintype "bidirectional+no_connect"))
     (pad "11" smd rect (at -2.1 11.2962) (size 1 2.45) (layers "F.Cu" "F.Paste" "F.Mask")
-      (net 10 "unconnected-(DWM1-GPIO4{slash}EXTPA-Pad11)") (pinfunction "GPIO4/EXTPA") (pintype "bidirectional+no_connect"))
+      (net 10 "Net-(D2-A)") (pinfunction "GPIO4/EXTPA") (pintype "bidirectional"))
     (pad "12" smd rect (at -0.7 11.2962) (size 1 2.45) (layers "F.Cu" "F.Paste" "F.Mask")
       (net 11 "unconnected-(DWM1-GPIO3{slash}TXLED-Pad12)") (pinfunction "GPIO3/TXLED") (pintype "bidirectional+no_connect"))
@@
     )
   )
-  (gr_rect (start 109.22 50.8) (end 152.4 81.28)
+  (footprint "LED_SMD:LED_0805_2012Metric_Pad1.15x1.40mm_HandSolder" (layer "F.Cu")
+    (at 149.86 81.28 -90)
+    (descr "LED SMD 0805 (2012 Metric), square (rectangular) end terminal, IPC_7351 nominal, (Body size source: https://docs.google.com/spreadsheets/d/1BsfQQcO9C6DZCsRaXUlFlo91Tg2WpOkGARC1WS5S8t0/edit?usp=sharing), generated with kicad-footprint-generator")
+    (tags "LED handsolder")
+    (property "Sheetfile" "keychain.kicad_sch")
+    (property "Sheetname" "")
+    (property "ki_description" "Light emitting diode")
+    (property "ki_keywords" "LED diode")
+    (attr smd)
+    (fp_text reference "D2" (at 0 -1.65 90) (layer "F.SilkS")
+        (effects (font (size 1 1) (thickness 0.15)))
+    )
+    (fp_text value "LED" (at 0 1.65 90) (layer "F.Fab")
+        (effects (font (size 1 1) (thickness 0.15)))
+    )
+    (fp_text user "${REFERENCE}" (at 0 0 90) (layer "F.Fab")
+        (effects (font (size 0.5 0.5) (thickness 0.08)))
+    )
+    (fp_line (start -1.86 -0.96) (end -1.86 0.96)
+      (stroke (width 0.12) (type solid)) (layer "F.SilkS"))
+    (fp_line (start -1.86 0.96) (end 1 0.96)
+      (stroke (width 0.12) (type solid)) (layer "F.SilkS"))
+    (fp_line (start 1 -0.96) (end -1.86 -0.96)
+      (stroke (width 0.12) (type solid)) (layer "F.SilkS"))
+    (fp_line (start -1.85 -0.95) (end 1.85 -0.95)
+      (stroke (width 0.05) (type solid)) (layer "F.CrtYd"))
+    (fp_line (start -1.85 0.95) (end -1.85 -0.95)
+      (stroke (width 0.05) (type solid)) (layer "F.CrtYd"))
+    (fp_line (start 1.85 -0.95) (end 1.85 0.95)
+      (stroke (width 0.05) (type solid)) (layer "F.CrtYd"))
+    (fp_line (start 1.85 0.95) (end -1.85 0.95)
+      (stroke (width 0.05) (type solid)) (layer "F.CrtYd"))
+    (fp_line (start -1 -0.3) (end -1 0.6)
+      (stroke (width 0.1) (type solid)) (layer "F.Fab"))
+    (fp_line (start -1 0.6) (end 1 0.6)
+      (stroke (width 0.1) (type solid)) (layer "F.Fab"))
+    (fp_line (start -0.7 -0.6) (end -1 -0.3)
+      (stroke (width 0.1) (type solid)) (layer "F.Fab"))
+    (fp_line (start 1 -0.6) (end -0.7 -0.6)
+      (stroke (width 0.1) (type solid)) (layer "F.Fab"))
+    (fp_line (start 1 0.6) (end 1 -0.6)
+      (stroke (width 0.1) (type solid)) (layer "F.Fab"))
+    (pad "1" smd roundrect (at -1.025 0 270) (size 1.15 1.4) (layers "F.Cu" "F.Paste" "F.Mask") (roundrect_rratio 0.217391)
+      (net 2 "GND") (pinfunction "K") (pintype "passive"))
+    (pad "2" smd roundrect (at 1.025 0 270) (size 1.15 1.4) (layers "F.Cu" "F.Paste" "F.Mask") (roundrect_rratio 0.217391)
+      (net 10 "Net-(D2-A)") (pinfunction "A") (pintype "passive"))
+    (model "${KICAD6_3DMODEL_DIR}/LED_SMD.3dshapes/LED_0805_2012Metric.wrl"
+      (offset (xyz 0 0 0))
+      (scale (xyz 1 1 1))
+      (rotate (xyz 0 0 0))
+    )
+  )
+  (gr_rect (start 109.22 53.34) (end 152.4 83.82)
     (stroke (width 0.1) (type default)) (fill none) (layer "Edge.Cuts"))
   (gr_text "Keychain PCB\n2024-03-19\nTeam 17" (at 124.46 53.34) (layer "F.SilkS")
@@
   )
   (dimension (type aligned) (layer "Dwgs.User")
-    (pts (xy 152.4 81.28) (xy 109.22 81.28))
+    (pts (xy 152.4 83.82) (xy 109.22 83.82))
     (height -2.54)
-    (gr_text "43.1800 mm" (at 130.81 82.67) (layer "Dwgs.User")
+    (gr_text "43.1800 mm" (at 130.81 85.21) (layer "Dwgs.User")
       (effects (font (size 1 1) (thickness 0.15)))
     )
@@
   (segment (start 129.54 76.2) (end 124.46 71.12) (width 0.254) (layer "B.Cu") (net 6))
   (segment (start 141.513 76.295199) (end 144.78 73.028199) (width 0.254) (layer "B.Cu") (net 6))
+  (segment (start 128.025 82.305) (end 149.86 82.305) (width 0.254) (layer "F.Cu") (net 10))
+  (segment (start 126.22 80.5) (end 128.025 82.305) (width 0.254) (layer "F.Cu") (net 10))
+  (segment (start 126.22 78.135) (end 126.22 80.5) (width 0.254) (layer "F.Cu") (net 10))
   (segment (start 138.1482 79.367) (end 143.623264 79.367) (width 0.254) (layer "F.Cu") (net 15))
   (segment (start 143.623264 79.367) (end 141.726264 77.47) (width 0.254) (layer "F.Cu") (net 15))

Commit message: generated week 3 gerbers
Other:
- board text added: "Keychain PCB V2 2024-03-19 Team 17"
- board text removed: "Keychain PCB 2024-03-19 Team 17"
Changed lines of the file:
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@@
       (plot_on_all_layers_selection 0x0000000_00000000)
       (disableapertmacros false)
-      (usegerberextensions false)
-      (usegerberattributes true)
+      (usegerberextensions true)
+      (usegerberattributes false)
       (usegerberadvancedattributes true)
-      (creategerberjobfile true)
+      (creategerberjobfile false)
       (dashed_line_dash_ratio 12.000000)
       (dashed_line_gap_ratio 3.000000)
@@
       (outputformat 1)
       (mirror false)
-      (drillshape 1)
+      (drillshape 0)
       (scaleselection 1)
-      (outputdirectory "")
+      (outputdirectory "v2 gerbers/")
     )
   )
@@
     (fp_line (start 1 0.625) (end -1 0.625)
       (stroke (width 0.1) (type solid)) (layer "F.Fab"))
-    (pad "1" smd roundrect (at -1 0 270) (size 1.2 1.4) (layers "F.Cu" "F.Paste" "F.Mask") (roundrect_rratio 0.208333)
+    (pad "1" smd roundrect (at -1 0 270) (size 1.2 1.4) (layers "F.Cu" "F.Paste" "F.Mask") (roundrect_rratio 0.2083333333)
       (net 2 "GND") (pintype "passive"))
-    (pad "2" smd roundrect (at 1 0 270) (size 1.2 1.4) (layers "F.Cu" "F.Paste" "F.Mask") (roundrect_rratio 0.208333)
+    (pad "2" smd roundrect (at 1 0 270) (size 1.2 1.4) (layers "F.Cu" "F.Paste" "F.Mask") (roundrect_rratio 0.2083333333)
       (net 19 "/interrupt") (pintype "passive"))
     (model "${KICAD6_3DMODEL_DIR}/Resistor_SMD.3dshapes/R_0805_2012Metric.wrl"
@@
     (fp_line (start 3.81 2.88) (end 3.81 -2.92)
       (stroke (width 0.1) (type solid)) (layer "F.Fab"))
-    (pad "1" thru_hole roundrect (at 0 0) (size 1.74 2.19) (drill 1.19) (layers "*.Cu" "*.Mask") (roundrect_rratio 0.143678)
+    (pad "1" thru_hole roundrect (at 0 0) (size 1.74 2.19) (drill 1.19) (layers "*.Cu" "*.Mask") (roundrect_rratio 0.1436781609)
       (net 2 "GND") (pinfunction "Pin_1") (pintype "passive"))
     (pad "2" thru_hole oval (at 2.54 0) (size 1.74 2.19) (drill 1.19) (layers "*.Cu" "*.Mask")
@@
     (fp_line (start 5.72 10.18) (end -3.18 10.18)
       (stroke (width 0.1) (type solid)) (layer "F.Fab"))
-    (pad "1" thru_hole roundrect (at 0 0) (size 1.7 1.7) (drill 1) (layers "*.Cu" "*.Mask") (roundrect_rratio 0.147059)
+    (pad "1" thru_hole roundrect (at 0 0) (size 1.7 1.7) (drill 1) (layers "*.Cu" "*.Mask") (roundrect_rratio 0.1470588235)
       (net 17 "/MISO") (pinfunction "MISO") (pintype "passive"))
     (pad "2" thru_hole circle (at 2.54 0) (size 1.7 1.7) (drill 1) (layers "*.Cu" "*.Mask")
@@
     (fp_line (start 1 0.625) (end -1 0.625)
       (stroke (width 0.1) (type solid)) (layer "F.Fab"))
-    (pad "1" smd roundrect (at -1.0375 0) (size 1.175 1.45) (layers "F.Cu" "F.Paste" "F.Mask") (roundrect_rratio 0.212766)
+    (pad "1" smd roundrect (at -1.0375 0) (size 1.175 1.45) (layers "F.Cu" "F.Paste" "F.Mask") (roundrect_rratio 0.2127659574)
       (net 1 "Net-(J3-Pin_2)") (pintype "passive"))
-    (pad "2" smd roundrect (at 1.0375 0) (size 1.175 1.45) (layers "F.Cu" "F.Paste" "F.Mask") (roundrect_rratio 0.212766)
+    (pad "2" smd roundrect (at 1.0375 0) (size 1.175 1.45) (layers "F.Cu" "F.Paste" "F.Mask") (roundrect_rratio 0.2127659574)
       (net 2 "GND") (pintype "passive"))
     (model "${KICAD6_3DMODEL_DIR}/Capacitor_SMD.3dshapes/C_0805_2012Metric.wrl"
@@
     (fp_line (start 1 0.625) (end -1 0.625)
       (stroke (width 0.1) (type solid)) (layer "F.Fab"))
-    (pad "1" smd roundrect (at -1 0) (size 1.2 1.4) (layers "F.Cu" "F.Paste" "F.Mask") (roundrect_rratio 0.208333)
+    (pad "1" smd roundrect (at -1 0) (size 1.2 1.4) (layers "F.Cu" "F.Paste" "F.Mask") (roundrect_rratio 0.2083333333)
       (net 3 "+3.3V") (pintype "passive"))
-    (pad "2" smd roundrect (at 1 0) (size 1.2 1.4) (layers "F.Cu" "F.Paste" "F.Mask") (roundrect_rratio 0.208333)
+    (pad "2" smd roundrect (at 1 0) (size 1.2 1.4) (layers "F.Cu" "F.Paste" "F.Mask") (roundrect_rratio 0.2083333333)
       (net 6 "/RST") (pintype "passive"))
     (model "${KICAD6_3DMODEL_DIR}/Resistor_SMD.3dshapes/R_0805_2012Metric.wrl"
@@
     (fp_line (start 1 0.625) (end -1 0.625)
       (stroke (width 0.1) (type solid)) (layer "F.Fab"))
-    (pad "1" smd roundrect (at -1.0375 0) (size 1.175 1.45) (layers "F.Cu" "F.Paste" "F.Mask") (roundrect_rratio 0.212766)
+    (pad "1" smd roundrect (at -1.0375 0) (size 1.175 1.45) (layers "F.Cu" "F.Paste" "F.Mask") (roundrect_rratio 0.2127659574)
       (net 3 "+3.3V") (pintype "passive"))
-    (pad "2" smd roundrect (at 1.0375 0) (size 1.175 1.45) (layers "F.Cu" "F.Paste" "F.Mask") (roundrect_rratio 0.212766)
+    (pad "2" smd roundrect (at 1.0375 0) (size 1.175 1.45) (layers "F.Cu" "F.Paste" "F.Mask") (roundrect_rratio 0.2127659574)
       (net 2 "GND") (pintype "passive"))
     (model "${KICAD6_3DMODEL_DIR}/Capacitor_SMD.3dshapes/C_0805_2012Metric.wrl"
@@
     (fp_line (start 1 0.6) (end 1 -0.6)
       (stroke (width 0.1) (type solid)) (layer "F.Fab"))
-    (pad "1" smd roundrect (at -1.025 0 270) (size 1.15 1.4) (layers "F.Cu" "F.Paste" "F.Mask") (roundrect_rratio 0.217391)
+    (pad "1" smd roundrect (at -1.025 0 270) (size 1.15 1.4) (layers "F.Cu" "F.Paste" "F.Mask") (roundrect_rratio 0.2173913043)
       (net 2 "GND") (pinfunction "K") (pintype "passive"))
-    (pad "2" smd roundrect (at 1.025 0 270) (size 1.15 1.4) (layers "F.Cu" "F.Paste" "F.Mask") (roundrect_rratio 0.217391)
+    (pad "2" smd roundrect (at 1.025 0 270) (size 1.15 1.4) (layers "F.Cu" "F.Paste" "F.Mask") (roundrect_rratio 0.2173913043)
       (net 10 "Net-(D2-A)") (pinfunction "A") (pintype "passive"))
     (model "${KICAD6_3DMODEL_DIR}/LED_SMD.3dshapes/LED_0805_2012Metric.wrl"
@@
   (gr_rect (start 109.22 53.34) (end 152.4 83.82)
     (stroke (width 0.1) (type default)) (fill none) (layer "Edge.Cuts"))
-  (gr_text "Keychain PCB\n2024-03-19\nTeam 17" (at 124.46 53.34) (layer "F.SilkS")
+  (gr_text "Keychain PCB V2\n2024-03-19\nTeam 17" (at 124.46 53.34) (layer "F.SilkS")
     (effects (font (size 0.5 0.5) (thickness 0.125)) (justify left bottom))
   )

Commit message: dish pcb updated
Parts:
- removed D2: LED, LED_SMD:LED_0805_2012Metric_Pad1.15x1.40mm_HandSolder
- removed J2: AVR-ISP-6, Connector_IDC:IDC-Header_2x03_P2.54mm_Vertical
- removed R1: 100, Resistor_SMD:R_0805_2012Metric_Pad1.20x1.40mm_HandSolder
- removed U3: LM1117MP-3.3, Package_TO_SOT_SMD:SOT-223-3_TabPin2
- added C1: 1uF, Capacitor_SMD:C_0805_2012Metric_Pad1.18x1.45mm_HandSolder, F.Cu at (136.1, 86.4)
- added C4: 10uF, Capacitor_SMD:C_0805_2012Metric_Pad1.18x1.45mm_HandSolder, F.Cu at (140.7, 83.8)
- added J1: Conn_01x05, Connector_Molex:Molex_KK-254_AE-6410-05A_1x05_P2.54mm_Vertical, F.Cu at (137.2, 58.4)
- added REF**: BAT_BU2032SM-HD-G, BU2032SM_HD_G:BAT_BU2032SM-HD-G, F.Cu at (111.8, 70.5)
- added Y1: 16MHz, Crystal:Crystal_HC49-U_Vertical, F.Cu at (131.9, 91.4)
- C2, C3: value 10uF -> 22p
- J3: value Vin -> AVR-ISP-6; footprint Connector_Molex:Molex_KK-254_AE-6410-02A_1x02_P2.54mm_Vertical -> Connector_IDC:IDC-Header_2x03_P2.54mm_Vertical
- U1: value ATtiny84A-SS -> ATmega328-A; footprint Package_SO:SOIC-14_3.9x8.7mm_P1.27mm -> Package_QFP:TQFP-32_7x7mm_P0.8mm
- moved J3 42.6 mm to (154.9, 88.9), turned to -90 degrees
- moved D1 36.5 mm to (140.6, 94.0), turned to 0 degrees
- moved R3 31.3 mm to (140.7, 88.9)
- moved C2 24.1 mm to (133.6, 81.3), turned to 180 degrees
- moved DWM1 20.5 mm to (148.6, 69.4)
- moved C3 19.8 mm to (125.5, 81.3), turned to 180 degrees
- moved U1 12.3 mm to (131.7, 68.6), turned to 180 degrees
Connections:
- C2 pad 1: Net-(J3-Pin_2) -> Net-(U1-XTAL2/PB7)
- C3 pad 1: +3.3V -> Net-(U1-XTAL1/PB6)
- DWM1 pad 11: Net-(D2-A) -> unconnected-(DWM1-GPIO4/EXTPA-Pad11)
- DWM1 pad 22: /interrupt -> unconnected-(DWM1-IRQ/GPIO8-Pad22)
- DWM1 pad 3: /RST -> /RESET
- J3 pad 1: GND -> /MISO
- J3 pad 2: Net-(J3-Pin_2) -> Net-(D1-A)
- R3 pad 2: /RST -> /RESET
- U1 pad 1: +3.3V -> unconnected-(U1-PD3-Pad1)
- U1 pad 14: GND -> unconnected-(U1-PB2-Pad14)
- U1 pad 3: unconnected-(U1-XTAL2/PB1-Pad3) -> GND
- U1 pad 4: /RST -> +3.3V
- U1 pad 5: unconnected-(U1-PB2-Pad5) -> GND
- U1 pad 6: /Csn -> +3.3V
- U1 pad 7: /MOSI -> Net-(U1-XTAL1/PB6)
- U1 pad 8: /MISO -> Net-(U1-XTAL2/PB7)
- U1 pad 9: /SCK -> unconnected-(U1-PD5-Pad9)
Routing:
- net /RESET: track 0.00 -> 64.0 mm, vias 0 -> 2
- net /Csn: track 15.2 -> 75.7 mm, vias 0 -> 2
- net /MOSI: track 28.6 -> 85.1 mm, vias 2 -> 4
- net /SCK: track 39.3 -> 95.3 mm, vias 0 -> 4
- net +3.3V: track 65.4 -> 113.8 mm, vias 4 -> 6
- net /MISO: track 38.0 -> 84.5 mm, vias 2 -> 7
- net /RST: track 42.8 -> 0.00 mm, vias 4 -> 0
- net Net-(U1-XTAL1/PB6): track 0.00 -> 36.9 mm, vias 0 -> 3
- net Net-(U1-XTAL2/PB7): track 0.00 -> 33.7 mm, vias 0 -> 2
- net Net-(D2-A): track 26.8 -> 0.00 mm
- net Net-(J3-Pin_2): track 19.0 -> 0.00 mm
- net GND: track 0.00 -> 13.9 mm, vias 0 -> 3
- net /interrupt: track 7.23 -> 0.00 mm
- net Net-(D1-A): track 8.67 -> 13.8 mm
Other:
- board size 43.2 x 30.5 mm -> 63.5 x 45.7 mm
- board text added: "keychain PCB V3 Team17"
- board text removed: "Keychain PCB V2 2024-03-19 Team 17"
