File: pcb/keychain/keychain.kicad_sch (KiCad schematic)
At the start: 10 parts, among them J2 AVR-ISP-6, J3 Vin, U1 ATtiny84A-SS, U3 LM1117MP-3.3

Commit message: update pcb
Parts:
- added D2: LED, LED_SMD:LED_0805_2012Metric_Pad1.15x1.40mm_HandSolder, symbol Device:LED
Connections:
- net GND: now also D2.1 (K)
- net at DWM1.11 (GPIO4/EXTPA): now also D2.2 (A)
- no-connect marks 16 -> 15
Changed lines of the file:
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@@
   (no_connect (at 68.58 88.9))
   (no_connect (at 76.2 158.75))
-  (no_connect (at 68.58 86.36))
   (no_connect (at 76.2 153.67))
   (no_connect (at 76.2 176.53))
@@
     (stroke (width 0) (type default))
   )
+  (wire (pts (xy 91.44 87.63) (xy 91.44 90.17))
+    (stroke (width 0) (type default))
+  )
   (wire (pts (xy 13.97 76.2) (xy 22.86 76.2))
     (stroke (width 0) (type default))
@@
     (stroke (width 0) (type default))
   )
+  (wire (pts (xy 76.2 86.36) (xy 77.47 87.63))
+    (stroke (width 0) (type default))
+  )
   (wire (pts (xy 76.2 166.37) (xy 96.52 166.37))
     (stroke (width 0) (type default))
@@
     (stroke (width 0) (type default))
   )
+  (wire (pts (xy 85.09 87.63) (xy 91.44 87.63))
+    (stroke (width 0) (type default))
+  )
   (wire (pts (xy 68.58 66.04) (xy 90.17 66.04))
     (stroke (width 0) (type default))
@@
   )
   (wire (pts (xy 81.28 53.34) (xy 81.28 55.88))
+    (stroke (width 0) (type default))
+  )
+  (wire (pts (xy 68.58 86.36) (xy 76.2 86.36))
     (stroke (width 0) (type default))
   )
@@
         (path "/ad21d4e4-60ce-4072-adeb-1aa1f99c7ef4"
           (reference "D1") (unit 1)
+        )
+      )
+    )
+  )
+  (symbol (lib_id "power:GND") (at 91.44 90.17 0) (unit 1)
+    (in_bom yes) (on_board yes) (dnp no) (fields_autoplaced)
+    (property "Reference" "#PWR07" (at 91.44 96.52 0)
+      (effects (font (size 1.27 1.27)) hide)
+    )
+    (property "Value" "GND" (at 91.44 95.25 0)
+      (effects (font (size 1.27 1.27)))
+    )
+    (property "Footprint" "" (at 91.44 90.17 0)
+      (effects (font (size 1.27 1.27)) hide)
+    )
+    (property "Datasheet" "" (at 91.44 90.17 0)
+      (effects (font (size 1.27 1.27)) hide)
+    )
+    (pin "1")
+    (instances
+      (project "keychain"
+        (path "/ad21d4e4-60ce-4072-adeb-1aa1f99c7ef4"
+          (reference "#PWR07") (unit 1)
         )
       )
@@
         )
       )
+    )
+  )
+  (symbol (lib_id "Device:LED") (at 81.28 87.63 180) (unit 1)
+    (in_bom yes) (on_board yes) (dnp no) (fields_autoplaced)
+    (property "Reference" "D2" (at 82.8675 80.01 0)
+      (effects (font (size 1.27 1.27)))
+    )
+    (property "Value" "LED" (at 82.8675 82.55 0)
+      (effects (font (size 1.27 1.27)))
+    )
+    (property "Footprint" "LED_SMD:LED_0805_2012Metric_Pad1.15x1.40mm_HandSolder" (at 81.28 87.63 0)
+      (effects (font (size 1.27 1.27)) hide)
+    )
+    (property "Datasheet" "~" (at 81.28 87.63 0)
+      (effects (font (size 1.27 1.27)) hide)
+    )
+    (pin "1")
+    (pin "2")
+    (instances
+      (project "keychain"
+        (path "/ad21d4e4-60ce-4072-adeb-1aa1f99c7ef4"
+          (reference "D2") (unit 1)
+        )
+      )

Commit message: dish pcb updated
Parts:
- removed D2: LED, LED_SMD:LED_0805_2012Metric_Pad1.15x1.40mm_HandSolder, symbol Device:LED
- removed J2: AVR-ISP-6, Connector_IDC:IDC-Header_2x03_P2.54mm_Vertical, symbol Connector:AVR-ISP-6
- removed J3: Vin, Connector_Molex:Molex_KK-254_AE-6410-02A_1x02_P2.54mm_Vertical, symbol Connector_Generic:Conn_01x02
- removed R1: 100, Resistor_SMD:R_0805_2012Metric_Pad1.20x1.40mm_HandSolder, symbol Device:R
- removed U1: ATtiny84A-SS, Package_SO:SOIC-14_3.9x8.7mm_P1.27mm, symbol MCU_Microchip_ATtiny:ATtiny84A-SS
- removed U3: LM1117MP-3.3, Package_TO_SOT_SMD:SOT-223-3_TabPin2, symbol Regulator_Linear:LM1117MP-3.3
- added BT1: BU2032SM-HD-G, BU2032SM-HD-G:BAT_BU2032SM-HD-G, symbol BU2032SM-HD-G:BU2032SM-HD-G
- added C1: 1uF, Capacitor_SMD:C_0805_2012Metric_Pad1.18x1.45mm_HandSolder, symbol Device:C
- added C4: 10uF, Capacitor_SMD:C_0805_2012Metric_Pad1.18x1.45mm_HandSolder, symbol Device:C
- added J1: Conn_01x05, Connector_Molex:Molex_KK-254_AE-6410-05A_1x05_P2.54mm_Vertical, symbol Connector_Generic:Conn_01x05
- added J3: AVR-ISP-6, Connector_IDC:IDC-Header_2x03_P2.54mm_Vertical, symbol Connector:AVR-ISP-6
- added U1: ATmega328-A, Package_QFP:TQFP-32_7x7mm_P0.8mm, symbol MCU_Microchip_ATmega:ATmega328-A
- added Y1: 16MHz, Crystal:Crystal_HC49-U_Vertical, symbol Device:Crystal
- C2, C3: value 10uF -> 22p
Connections:
- net +3.3V: now also C1.2, C4.1, U1.18 (AVCC), U1.4 (VCC), U1.6 (VCC); no longer C3.1
- net Csn: now also J1.5 (Pin_5)
- net GND: now also BT1.-, C1.1, J3.6 (GND), U1.21 (GND), U1.3 (GND), U1.5 (GND)
- net MISO: now also J1.2 (Pin_2), J3.1 (MISO), U1.16 (PB4)
- net MOSI: now also J1.1 (Pin_1), J3.4 (MOSI), U1.15 (PB3)
- net SCK: now also J1.3 (Pin_3), J3.3 (SCK), U1.17 (PB5)
- net at C2.1: now also U1.8 (XTAL2/PB7), Y1.1
- net at D1.2 (A): now also J3.2 (VCC)
- net RST renamed RESET
- net RESET: now also J1.4 (Pin_4), J3.5 (~{RST}), U1.29 (~{RESET}/PC6)
- net interrupt: no longer names the net of DWM1.22 (IRQ/GPIO8)
- new net: BT1.+, C4.2
- new net: C3.1, U1.7 (XTAL1/PB6), Y1.2
- no-connect marks 15 -> 30
Other:
- note added: "Confirmation"
